File: kid-v2.brd (EAGLE design)
At the start: 30 x 110 mm, 103 parts, among them IC1 TL072D, IC13 LM404010, IC2 TL072D, IC3 LM13700M, IC5 TL072D, IC6 TL072D, IC7 TL072D, IC8 LM4040B10, IC9 TL331, Q1 pmp5201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

Commit message: Add files via upload
Updated silkscreen
Parts:
- moved R48 1.02 mm to (22.1, 37.6)
Other:
- board text added: "FANCYYYYY KID V.2"
